File: Hardware/GateMate_SoM/GateMate_SoM.kicad_sch (KiCad schematic)
At the start: 1 part, among them U1 CCGM1A1

Commit message: Schematics: Power supply
Parts:
- added C100, C95, C96, C99: 10uF, Capacitor_SMD:C_0402_1005Metric, symbol RA8M1:885012205092
- added C101, C102, C97, C98: 22uF, Capacitor_SMD:C_0805_2012Metric, symbol RA8M1:885012205092
- added J1: SODIMM-200_Split, symbol Connector:SODIMM-200_Split
- added L1, L2, L3, L4: 1uH, Inductor_SMD:L_0805_2012Metric, symbol Device:L
- added R17: 442k, Resistor_SMD:R_0402_1005Metric, symbol Device:R
- added R18, R20, R22, R23, R24: 100K, Resistor_SMD:R_0402_1005Metric, symbol Device:R
- added R19: 316k, Resistor_SMD:R_0402_1005Metric, symbol Device:R
- added R21: 150k, Resistor_SMD:R_0402_1005Metric, symbol Device:R
- added U4, U5, U6, U7: TPS62A02ADRL, Package_TO_SOT_SMD:SOT-563, symbol Regulator_Switching:TPS62A02ADRL
Connections:
- net GND: now reaches U1.A1 (GND), U1.A10 (GND), U1.A13 (GND), U1.A18 (GND), U1.A7 (GND), U1.B16 (GND), U1.C1 (GND), U1.E11 (GND), U1.E13 (GND), U1.E18 (GND), U1.E5 (GND), U1.E7 (GND), U1.E9 (GND), U1.F1 (GND), U1.F10 (GND), U1.F12 (GND), U1.F14 (GND), U1.F6 (GND), U1.F8 (GND), U1.G11 (GND), U1.G13 (GND), U1.G5 (GND), U1.G7 (GND), U1.G9 (GND), U1.H10 (GND), U1.H12 (GND), U1.H14 (GND), U1.H18 (GND), U1.H6 (GND), U1.H8 (GND), U1.J1 (GND), U1.J11 (GND), U1.J13 (GND), U1.J5 (GND), U1.J7 (GND), U1.J9 (GND), U1.K10 (GND), U1.K12 (GND), U1.K14 (GND), U1.K6 (GND), U1.K8 (GND), U1.L11 (GND), U1.L13 (GND), U1.L18 (GND), U1.L5 (GND), U1.L7 (GND), U1.L9 (GND), U1.M1 (GND), U1.M10 (GND), U1.M12 (GND), U1.M16 (GND), U1.M6 (GND), U1.M8 (GND), U1.N12 (GND), U1.N17 (GND), U1.N7 (GND), U1.N9 (GND), U1.P4 (GND), U1.P7 (GND), U1.P9 (GND), U1.R12 (GND), U1.R16 (GND), U1.T11 (GND), U1.T17 (GND), U1.T4 (GND), U1.U14 (GND), U1.U15 (GND), U1.U16 (GND), U1.V1 (GND), U1.V14 (GND), U1.V16 (GND), U1.V18 (GND), U1.V6 (GND), U1.V9 (GND)
- net GND: now also C100.1, C101.1, C102.1, C95.1, C96.1, C97.1, C98.1, C99.1, R18.1, R20.1, R22.1, R24.1, U4.1 (GND), U5.1 (GND), U6.1 (GND), U7.1 (GND)
- new net: R23.1, R24.2, U7.5 (FB)
- new net: L4.1, U7.2 (SW)
- new net: L1.1, U4.2 (SW)
- new net: R17.1, R18.2, U4.5 (FB)
- new net: L3.1, U6.2 (SW)
- new net: L2.1, U5.2 (SW)
- new net: R19.1, R20.2, U5.5 (FB)
- new net: R21.1, R22.2, U6.5 (FB)
- new net 1.2V: C102.2, L4.2, R23.2
- new net 1.5V: C101.2, L3.2, R21.2
- new net 1.5V_PG: U5.4 (EN), U6.6 (PG), U7.4 (EN)
- new net 2.5V: C98.2, L2.2, R19.2
- new net 3.3V: C97.2, L1.2, R17.2
- new net 5V: C100.2, C95.2, C96.2, C99.2, U4.3 (VIN), U5.3 (VIN), U6.3 (VIN), U7.3 (VIN)
- new net BB_PGOOD: U4.4 (EN), U6.4 (EN)
- no-connect marks 0 -> 3
Other:
- note added: "1.8A"
- note added: "POWER SUPPLY"
- note added: "PS 1.2V"
- note added: "PS 1.5V"
- note added: "PS 2.5V"
- note added: "PS 3.3V"
- note added: "R1=100k((1.2V/0.6V)-1)=100k"
- note added: "R1=100k((1.5V/0.6V)-1)=150k"
- note added: "R1=100k((2.5V/0.6V)-1)=317k"
- note added: "R1=100k((3.3V/0.6V)-1)=450k"
- moved on the sheet: U1A, U1B, U1C, U1D, U1E, U1F, U1G, U1H
